File: pcb-adr1399-vref.kicad_pcb (KiCad board)
At the start: 2 copper layers, 60 x 39 mm, 17 parts, among them J1 Barrel_Jack_Switch, J2 CT3151SP-2, J3 CT3151SP-0, U1 ADR1399, U2 LT1012

Commit message: Ordered P1B
Parts:
- added kibuzzard-61FB27BC: G***, kibuzzard-61FB27BC, F.Cu at (100.5, 94.5)
- moved kibuzzard-61E8B62B 2.50 mm to (115.5, 104.5)
- moved J2 1.03 mm to (113.5, 113.0)
- moved J3 1.03 mm to (113.5, 96.0)
- moved J1 1.00 mm to (80.0, 94.5)
Routing:
- net /VOUT: track 39.9 -> 38.1 mm
