File: pcb-adr1399-vref.kicad_sch (KiCad schematic)
At the start: 17 parts, among them J1 Barrel_Jack_Switch, J2 CT3151SP-2, J3 CT3151SP-0, U1 ADR1399, U2 LT1012

Commit message: Update pcb-adr1399-vref.kicad_sch
Other:
- title: Cover -> Cover test
Changed lines of the file:
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@@
   (paper "A4")
   (title_block
-    (title "Cover")
+    (title "Cover test")
     (date "%%date%%")
     (rev "%%version%%")
